File: GPRv2/docs/PWM/pcb/triangular/triangular.kicad_sch (KiCad schematic)
At the start: 27 parts, among them J1 Pote 100k (Bourns 3590), J2 12 V, J3 Salida, U1 TLC2274, U2 TLC2274

Commit message: GPRv2: PCB del generador de triangular terminado
- Esquematico: 2 TLC2274 repartidos por funcion (U1: integrador, Schmitt y
  sync; U2: 6 V y restador); las 3 unidades que sobran van como seguidor con
  la + a GND, asi mid no cruza la placa.
- SW1: llave palanca SPDT (LP-SW-213CI) de encendido en los 12 V, con LED
  rojo 5x5 (D2 + R17 2k2, ~4,7 mA). Se descarto el PULS-2I-RET: medido, su
  comun es un extremo de cada fila, no la pata del medio.
- JP1: puente de cable a 22,5 mm en la salida, antes de D1.
- triangular.pretty + fp-lib-table: huellas propias (llave a 4 mm con pads
  angostos, puente de 22,5 mm y el pulsador 8x8 por si se vuelve a usar).
- simular_kicad.py: detecta solo los operacionales que sobran, toma sq/tri/
  mid por etiqueta, simula la llave cerrada, el puente y el LED.
- PCB ruteado a una capa.

Co-Authored-By: Claude Opus 5.5 <noreply@anthropic.com>
Parts:
- added D2: LED rojo 5x5, LED_THT:LED_Rectangular_W5.0mm_H5.0mm, symbol Device:LED
- added JP1: Puente, triangular:Puente_Cable_P22.5mm, symbol Jumper:Jumper_2_Bridged
- added R17: 2k2, Resistor_THT:R_Axial_DIN0207_L6.3mm_D2.5mm_P10.16mm_Horizontal, symbol Device:R
- added SW1: LP-SW-213CI, triangular:SW_Palanca_SPDT_P4mm, symbol Switch:SW_SPDT
Connections:
- net +12V: now also R17.1, SW1.3 (C); no longer J2.1 (Pin_1)
- net GND: now also U1.12 (+), U2.10 (+), U2.12 (+), D2.1 (K)
- net mid: no longer U1.12 (+), U2.10 (+), U2.12 (+)
- net salida: now also JP1.2 (B); no longer R7.2, U2.7
- new net: JP1.1 (A), R7.2, U2.7
- new net: J2.1 (Pin_1), SW1.2 (B)
- new net: D2.2 (A), R17.2
- no-connect marks 0 -> 1
Other:
- note added: "U1D, U2C y U2D sobran: seguidores con la + a GND"
- note removed: "U1D, U2C y U2D sobran: seguidores con la entrada en mid"
